File: Adapterboard.kicad_pcb (KiCad board)
At the start: 2 copper layers, 100 x 100 mm, 78 parts, among them J101 reserve IO, J102 JTAG, J103 X, J104 Y, J105 Z, J106 TUNNEL_IN, J107 Power, J108 Piezzo XYZ, J109 U Preamp, J110 Tunnel_ADC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

Commit message: KiCad v7 update
Parts:
- moved U102 0.51 mm to (57.7, 131.4)
- turned J112 to 0 degrees
Connections:
- net /TUNNEL_IN_ADC renamed /TUNNEL_TO_ADC
Routing:
- net +5V: track 300.3 -> 296.1 mm
- net ESP32_CS1: track 66.4 -> 69.8 mm
- net Z-X: track 32.9 -> 29.6 mm
Other:
- board text added: "Socket ADC"
- board text added: "Socket DAC X"
- board text added: "Socket DAC Y"
- board text added: "Socket DAC Z"
- board text added: "Socket ESP32 DevKit"
- board text added: "Tunnel Current ADC"
- board text added: "to ADC"
- board text removed: "Tunnel to ADC"

Commit message: ESP 3D added
Changed lines of the file:
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@@
   )
   (paper "A4")
+  (title_block
+    (title "500EUR RTM Adapterboard")
+    (date "2023-06-20")
+    (company "Universität Regesburg")
+    (comment 1 "Peter Dirnhofer")
+  )
   (layers
     (0 "F.Cu" signal)
@@
     (property "ki_keywords" "R res resistor")
     (attr through_hole)
-    (fp_text reference "R125" (at 1.905 1.905) (layer "F.SilkS")
+    (fp_text reference "R125" (at 2.032 2.667) (layer "F.SilkS")
         (effects (font (size 1 1) (thickness 0.15)))
     )
@@
     (property "ki_keywords" "LED diode")
     (attr through_hole)
-    (fp_text reference "D102" (at 1.366487 -3.175 180) (layer "F.SilkS")
+    (fp_text reference "D102" (at 4.45 0 -90) (layer "F.SilkS")
         (effects (font (size 1 1) (thickness 0.15)))
     )
@@
     (property "ki_keywords" "R res resistor")
     (attr through_hole)
-    (fp_text reference "R126" (at 1.905 1.905) (layer "F.SilkS")
+    (fp_text reference "R126" (at 1.905 2.794) (layer "F.SilkS")
         (effects (font (size 1 1) (thickness 0.15)))
     )
@@
     (property "ki_keywords" "diode Schottky")
     (attr through_hole)
-    (fp_text reference "D108" (at 9.525 -2.54) (layer "F.SilkS")
+    (fp_text reference "D108" (at 5.461 2.467) (layer "F.SilkS")
         (effects (font (size 1 1) (thickness 0.15)))
     )
@@
     (property "ki_keywords" "dual opamp")
     (attr through_hole)
-    (fp_text reference "U101" (at 5.705 -3.185 90) (layer "F.SilkS")
+    (fp_text reference "U101" (at 3.673 2.657 90) (layer "F.SilkS")
         (effects (font (size 1 1) (thickness 0.15)))
     )
@@
     (property "ki_keywords" "diode Schottky")
     (attr through_hole)
-    (fp_text reference "D109" (at 5.08 -2.47) (layer "F.SilkS")
+    (fp_text reference "D109" (at 5.08 -2.286) (layer "F.SilkS")
         (effects (font (size 1 1) (thickness 0.15)))
     )
@@
     (property "ki_keywords" "cap capacitor")
     (attr through_hole)
-    (fp_text reference "C104" (at 1.25 1.905 270) (layer "F.SilkS")
+    (fp_text reference "C104" (at 6.711 0 270) (layer "F.SilkS")
         (effects (font (size 1 1) (thickness 0.15)))
     )
@@
     (property "ki_keywords" "LED diode")
     (attr through_hole)
-    (fp_text reference "D101" (at 1.275 -3.175) (layer "F.SilkS")
+    (fp_text reference "D101" (at -1.773 -0.127 90) (layer "F.SilkS")
         (effects (font (size 1 1) (thickness 0.15)))
     )
@@
     (property "ki_keywords" "diode Schottky")
     (attr through_hole)
-    (fp_text reference "D107" (at 10.16 -1.905) (layer "F.SilkS")
+    (fp_text reference "D107" (at 5.461 2.413) (layer "F.SilkS")
         (effects (font (size 1 1) (thickness 0.15)))
     )
@@
     (pad "J3-19" thru_hole circle locked (at 12.7 25.96 180) (size 1.56 1.56) (drill 1.04) (layers "*.Cu" "*.Mask")
       (net 87 "unconnected-(U103-CLK-PadJ3-19)") (pinfunction "CLK") (pintype "input+no_connect"))
+    (model "${KICAD7_3DMODEL_DIR}/ESP32_Dev_kit/ESP32-WROOM-32D-Assembly.STEP"
+      (offset (xyz 0 -3.5 7))
+      (scale (xyz 1 1 1))
+      (rotate (xyz 90 180 180))
+    )
   )
   (footprint "Resistor_THT:R_Axial_DIN0207_L6.3mm_D2.5mm_P10.16mm_Horizontal" (layer "F.Cu")
@@
     (property "ki_keywords" "dual opamp")
     (attr through_hole)
-    (fp_text reference "U105" (at 5.705 -3.185 90) (layer "F.SilkS")
+    (fp_text reference "U105" (at 3.8 2.784 90) (layer "F.SilkS")
         (effects (font (size 1 1) (thickness 0.15)))
     )
@@
     (property "ki_keywords" "diode Schottky")
     (attr through_hole)
-    (fp_text reference "D105" (at 10.16 -1.905) (layer "F.SilkS")
+    (fp_text reference "D105" (at 5.207 2.286) (layer "F.SilkS")
         (effects (font (size 1 1) (thickness 0.15)))
     )
@@
     (property "ki_keywords" "cap capacitor")
     (attr through_hole)
-    (fp_text reference "C109" (at 1.25 2.54 90) (layer "F.SilkS")
+    (fp_text reference "C109" (at 6.33 0.254 90) (layer "F.SilkS")
         (effects (font (size 1 1) (thickness 0.15)))
     )
@@
     (effects (font (size 0.8 0.7) (thickness 0.15)))
   )
-  (gr_text "IO04" (at 99.695 53.34) (layer "F.SilkS")
+  (gr_text "IO04" (at 99.822 55.118) (layer "F.SilkS")
     (effects (font (size 1 1) (thickness 0.15)))
   )
-  (gr_text "IO17" (at 94.615 53.34) (layer "F.SilkS")
+  (gr_text "IO17" (at 94.615 55.118) (layer "F.SilkS")
     (effects (font (size 1 1) (thickness 0.15)))
   )
