File: Adapterboard.kicad_sch (KiCad schematic)
At the start: 78 parts, among them J101 reserve IO, J102 JTAG, J103 X, J104 Y, J105 Z, J106 TUNNEL_IN, J107 Power, J108 Piezzo XYZ, J109 U Preamp, J110 Tunnel_ADC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

Commit message: KiCad v7 update
Parts:
- J101, J107: symbol Connector:Conn_01x04_Male -> Connector:Conn_01x04_Pin
- J102, J108: symbol Connector:Conn_01x05_Male -> Connector:Conn_01x05_Pin
- J103, J104, J105, J111, J112, J113: symbol Connector:Conn_01x01_Female -> Connector:Conn_01x01_Socket
- J109: symbol Connector:Conn_01x03_Male -> Connector:Conn_01x03_Pin
- J110: symbol Connector:Conn_01x02_Male -> Connector:Conn_01x02_Socket
Connections:
- net TUNNEL_IN_ADC renamed TUNNEL_TO_ADC
Changed lines of the file:
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@@
   (junction (at 211.455 228.6) (diameter 0) (color 0 0 0 0)
   )
+  (junction (at 257.81 98.425) (diameter 0) (color 0 0 0 0)
+  )
   (junction (at 314.96 46.355) (diameter 0) (color 0 0 0 0)
   )
@@
   (junction (at 269.875 36.83) (diameter 0) (color 0 0 0 0)
   )
-  (junction (at 257.81 98.425) (diameter 0) (color 0 0 0 0)
-  )
   (junction (at 175.895 170.18) (diameter 0) (color 0 0 0 0)
   )
@@
     (stroke (width 0) (type default))
   )
+  (wire (pts (xy 269.24 100.965) (xy 316.23 100.965))
+    (stroke (width 0) (type default))
+  )
   (wire (pts (xy 43.815 206.375) (xy 43.815 208.915))
     (stroke (width 0) (type default))
@@
     (stroke (width 0) (type default))
   )
-  (wire (pts (xy 257.81 98.425) (xy 287.655 98.425))
-    (stroke (width 0) (type default))
-  )
   (wire (pts (xy 284.48 203.2) (xy 286.385 203.2))
     (stroke (width 0) (type default))
@@
     (stroke (width 0) (type default))
   )
-  (wire (pts (xy 251.46 98.425) (xy 257.81 98.425))
-    (stroke (width 0) (type default))
-  )
   (wire (pts (xy 128.27 48.26) (xy 133.35 48.26))
     (stroke (width 0) (type default))
@@
     (stroke (width 0) (type default))
   )
+  (wire (pts (xy 257.81 98.425) (xy 316.23 98.425))
+    (stroke (width 0) (type default))
+  )
   (wire (pts (xy 34.29 59.69) (xy 39.37 59.69))
     (stroke (width 0) (type default))
@@
     (stroke (width 0) (type default))
   )
-  (wire (pts (xy 287.655 100.965) (xy 269.24 100.965))
-    (stroke (width 0) (type default))
-  )
   (wire (pts (xy 267.97 53.975) (xy 273.05 53.975))
     (stroke (width 0) (type default))
@@
     (stroke (width 0) (type default))
   )
+  (wire (pts (xy 251.46 98.425) (xy 257.81 98.425))
+    (stroke (width 0) (type default))
+  )
   (wire (pts (xy 175.895 170.18) (xy 175.895 181.61))
     (stroke (width 0) (type default))
@@
     (effects (font (size 1.27 1.27)) (justify left bottom))
   )
-  (label "TUNNEL_IN_ADC" (at 273.05 98.425 0) (fields_autoplaced)
+  (label "TUNNEL_TO_ADC" (at 273.05 98.425 0) (fields_autoplaced)
     (effects (font (size 1.27 1.27)) (justify left bottom))
   )
@@
     )
   )
-  (symbol (lib_name "Mikroe-Socket_1") (lib_id "mikroe:Mikroe-Socket") (at 53.34 118.11 0) (unit 1)
+  (symbol (lib_id "mikroe:Mikroe-Socket") (at 53.34 118.11 0) (unit 1)
     (in_bom yes) (on_board yes) (dnp no)
     (property "Reference" "U102" (at 52.07 111.76 0)
@@
       (effects (font (size 1.27 1.27)))
     )
-    (property "Footprint" "Mikroe:Mikroe_Socket_DAC_2_Click" (at 54.61 101.6 0)
-      (effects (font (size 1.27 1.27)) hide)
+    (property "Footprint" "Mikroe:Mikroe_Socket_DAC_2_Click" (at 54.61 101.6 0) (show_name)
+      (effects (font (size 1.27 1.27)))
     )
     (property "Datasheet" "" (at 52.07 110.49 0)
@@
     )
   )
-  (symbol (lib_name "Mikroe-Socket_3") (lib_id "mikroe:Mikroe-Socket") (at 307.975 113.665 0) (unit 1)
+  (symbol (lib_id "mikroe:Mikroe-Socket") (at 307.975 113.665 0) (unit 1)
     (in_bom yes) (on_board yes) (dnp no)
     (property "Reference" "U108" (at 306.705 107.315 0)
@@
       (effects (font (size 1.27 1.27)))
     )
-    (property "Footprint" "Mikroe:Mikroe_Socket_ADC_8_Click" (at 306.705 106.045 0)
-      (effects (font (size 1.27 1.27)) hide)
+    (property "Footprint" "Mikroe:Mikroe_Socket_ADC_8_Click" (at 306.705 106.045 0) (show_name)
+      (effects (font (size 1.27 1.27)))
     )
     (property "Datasheet" "" (at 306.705 106.045 0)
@@
     )
   )
-  (symbol (lib_id "Connector:Conn_01x01_Female") (at 175.26 110.49 270) (unit 1)
+  (symbol (lib_id "Connector:Conn_01x01_Socket") (at 175.26 110.49 270) (unit 1)
     (in_bom yes) (on_board yes) (dnp no)
     (property "Reference" "J105" (at 177.165 108.5849 90)
@@
     )
   )
-  (symbol (lib_id "Connector:Conn_01x04_Male") (at 27.305 43.18 0) (unit 1)
+  (symbol (lib_id "Connector:Conn_01x04_Pin") (at 27.305 43.18 0) (unit 1)
     (in_bom yes) (on_board yes) (dnp no)
     (property "Reference" "J101" (at 24.13 38.1 0)
@@
     )
   )
-  (symbol (lib_id "Connector:Conn_01x05_Male") (at 279.4 205.74 0) (unit 1)
+  (symbol (lib_id "Connector:Conn_01x05_Pin") (at 279.4 205.74 0) (unit 1)
     (in_bom yes) (on_board yes) (dnp no) (fields_autoplaced)
     (property "Reference" "J108" (at 280.035 194.945 0)
@@
     )
   )
-  (symbol (lib_id "Connector:Conn_01x05_Male") (at 29.21 64.77 0) (unit 1)
+  (symbol (lib_id "Connector:Conn_01x05_Pin") (at 29.21 64.77 0) (unit 1)
     (in_bom yes) (on_board yes) (dnp no) (fields_autoplaced)
     (property "Reference" "J102" (at 29.845 54.61 0)
@@
     )
   )
-  (symbol (lib_id "Connector:Conn_01x02_Male") (at 292.735 100.965 180) (unit 1)
+  (symbol (lib_id "Connector:Conn_01x02_Socket") (at 321.31 100.965 0) (mirror x) (unit 1)
     (in_bom yes) (on_board yes) (dnp no)
-    (property "Reference" "J110" (at 290.83 104.14 0)
+    (property "Reference" "J110" (at 325.12 97.155 0)
       (effects (font (size 1.27 1.27)))
     )
-    (property "Value" "Tunnel_ADC" (at 302.895 99.695 0)
+    (property "Value" "Tunnel_ADC" (at 327.66 100.965 0)
       (effects (font (size 1.27 1.27)))
     )
-    (property "Footprint" "Connector_PinHeader_2.54mm:PinHeader_1x02_P2.54mm_Vertical" (at 292.735 100.965 0)
+    (property "Footprint" "Connector_PinHeader_2.54mm:PinHeader_1x02_P2.54mm_Vertical" (at 321.31 100.965 0)
       (effects (font (size 1.27 1.27)) hide)
     )
-    (property "Datasheet" "~" (at 292.735 100.965 0)
+    (property "Datasheet" "~" (at 321.31 100.965 0)
       (effects (font (size 1.27 1.27)) hide)
     )
@@
     )
   )
-  (symbol (lib_id "Connector:Conn_01x01_Female") (at 332.74 46.355 180) (unit 1)
+  (symbol (lib_id "Connector:Conn_01x01_Socket") (at 332.74 46.355 180) (unit 1)
     (in_bom yes) (on_board yes) (dnp no)
     (property "Reference" "J112" (at 335.915 43.18 0)
@@
     )
   )
-  (symbol (lib_id "Connector:Conn_01x04_Male") (at 239.395 36.83 0) (unit 1)
+  (symbol (lib_id "Connector:Conn_01x04_Pin") (at 239.395 36.83 0) (unit 1)
     (in_bom yes) (on_board yes) (dnp no) (fields_autoplaced)
     (property "Reference" "J107" (at 240.03 28.575 0)
@@
     )
   )
-  (symbol (lib_id "Connector:Conn_01x01_Female") (at 370.205 67.945 180) (unit 1)
+  (symbol (lib_id "Connector:Conn_01x01_Socket") (at 370.205 67.945 180) (unit 1)
     (in_bom yes) (on_board yes) (dnp no)
     (property "Reference" "J113" (at 372.1101 69.85 0)
@@
     )
   )
-  (symbol (lib_id "Connector:Conn_01x01_Female") (at 53.34 110.49 270) (unit 1)
+  (symbol (lib_id "Connector:Conn_01x01_Socket") (at 53.34 110.49 270) (unit 1)
     (in_bom yes) (on_board yes) (dnp no)
     (property "Reference" "J103" (at 55.245 108.5849 90)
@@
     )
   )
-  (symbol (lib_id "Connector:Conn_01x01_Female") (at 114.3 110.49 270) (unit 1)
+  (symbol (lib_id "Connector:Conn_01x01_Socket") (at 114.3 110.49 270) (unit 1)
     (in_bom yes) (on_board yes) (dnp no)
     (property "Reference" "J104" (at 116.205 108.5849 90)
@@
     )
   )
-  (symbol (lib_id "Connector:Conn_01x03_Male") (at 267.335 64.77 0) (unit 1)
+  (symbol (lib_id "Connector:Conn_01x03_Pin") (at 267.335 64.77 0) (unit 1)
     (in_bom yes) (on_board yes) (dnp no)
     (property "Reference" "J109" (at 262.255 63.5 0)
@@
     )
   )
-  (symbol (lib_id "Connector:Conn_01x01_Female") (at 304.165 46.355 180) (unit 1)
+  (symbol (lib_id "Connector:Conn_01x01_Socket") (at 304.165 46.355 180) (unit 1)
     (in_bom yes) (on_board yes) (dnp no)
     (property "Reference" "J111" (at 306.07 43.815 0)

Commit message: ESP 3D added
Other:
- title: RTM Adapterboard -> 500EUR RTM Adapterboard
Changed lines of the file:
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@@
   (paper "A3")
   (title_block
-    (title "RTM Adapterboard")
-    (date "2023-02-27")
+    (title "500EUR RTM Adapterboard")
+    (date "2023-06-20")
     (rev "2.3")
     (company "Universität Regensburg")
